Commit message: make all parameters unique in robot1 for easy test interpretation

File: urdf/robot1.urdf (robot description, URDF)
Before this commit: robot robot1, 8 links, 7 joints
Joints:
- joint joint_a1: origin xyz=0 0 0.1 rpy=0 0 0 -> xyz=0 0 0.070 rpy=0 0 0

Commit message: make a2 positive for test robot 1

File: urdf/robot1.urdf (robot description, URDF)
Before this commit: robot robot1, 8 links, 7 joints
Joints:
- joint joint_a4: origin xyz=-0.05 0.1 0 rpy=0 0 0 -> xyz=0.05 0.1 0 rpy=0 0 0
